File: GPSmod.kicad_sch (KiCad schematic)
At the start: 6 parts, among them U1 AT2659, U2 ATGM336H-5N31

Commit message: added the GPS and finished Bluetooth antennas
Parts:
- removed C10: 0402, X7R, 100nF, easyeda:C0402, symbol EasyEDA:CL05B104KO5NNNC
- removed C13: 0402, C0G/NP0, 470pF, ±5%, easyeda:C0603, symbol EasyEDA:0603B471K500NT
- removed C19: 10uF, easyeda:C0603, symbol EasyEDA:CL10A106KP8NNNC
- removed L6: LQW15AN6N8G00D, easyeda:L0402, symbol EasyEDA:LQW15AN6N8G00D
- removed U1: AT2659, easyeda:DFN-6_L1.6-W1.0-P0.55-BL, symbol EasyEDA:AT2659
- removed U2: ATGM336H-5N31, easyeda:GPSM-SMD_ATGM336H-TR, symbol EasyEDA:ATGM336H-5N31
