File: Wtracker.kicad_sch (KiCad schematic)
At the start: 22 parts, among them IC1 RFX2401C, U2 ATGM336H-5N31, U3 ANT3216A063R2400A_C20619632, U4 NRF52840-QIAA-R

Commit message: worked on antenna of pcb
Parts:
- removed C1, C2, C5, C6: C, symbol Device:C
- removed C3: 1pF, symbol Device:C
- removed C4: 1.2pF, symbol Device:C
- removed L1: 4.7nH, symbol Device:L
- removed L2, L4: n/a, symbol Device:L
- removed L3: 15nH, symbol Device:L
- removed L5: 2.2nH, symbol Device:L
- removed U2: ATGM336H-5N31, easyeda:GPSM-SMD_ATGM336H-TR, symbol EasyEDA:ATGM336H-5N31
- removed U3: ANT3216A063R2400A_C20619632, easyeda:ANT-SMD_3P-L3.1-W1.6, symbol EasyEDA:ANT3216A063R2400A_C20619632
- added C1, C17, C18, C2: 12pF NP0 ±2%, 0402, easyeda:C0402, symbol EasyEDA:0402CG120J500NT
- added C11, C12, C7, C8: 100pF NP0 ±5%, 0402, easyeda:C0402, symbol EasyEDA:0402CG101J500NT
- added C14, C15: 1.0µF X7R ±10%, 0603, GRM18x, symbol GRM188Z71A475KE15D:GRM188Z71A475KE15D
- added C16: 4.7nF X7R ±10%, easyeda:C0402, symbol EasyEDA:CL05B104KO5NNNC
- added C4: 1.0pF NP0 ±5%, 0402, easyeda:C0402, symbol EasyEDA:0402CG101J500NT
- added C5: 100nF X7R ±10%, 0402, easyeda:C0402, symbol EasyEDA:CL05B104KO5NNNC
- added C6: 4.7uF X7R ±10%, 0603, GRM18x, symbol GRM188Z71A475KE15D:GRM188Z71A475KE15D
- added C9: 820pF NP0 ±5%, 0402, easyeda:C0402, symbol EasyEDA:CL05B104KO5NNNC
- added L1: 4.7nH ±5%, 0402, easyeda:L0402, symbol EasyEDA:LQP15MN4N7B02D
- added L2: 10µH, IDC≥50mA, 0603, easyeda:L0603, symbol EasyEDA:SDFL1608S100KTF
- added L4: 10µH, IDC≥80mA, 0603, easyeda:L0603, symbol EasyEDA:SDFL1608S100KTF
- added L5: 3.9nH ±5%, 0402, easyeda:L0402, symbol EasyEDA:LQG15HS2N2S02D
- added L7: ANT3216A063R2400A, easyeda:ANT-SMD_3P-L3.1-W1.6_ANT3216A063R2400A, symbol EasyEDA:ANT3216A063R2400A
- added X1: NX2016SA-32MHZ-STD-CZS-5, easyeda:OSC-SMD_4P-L2.0-W1.6-BL, symbol EasyEDA:NX2016SA-32MHZ-STD-CZS-5
- B1: footprint EasyEDA:BAT-TH_CR2032-BS-6-1 -> easyeda:BAT-TH_CR2032-BS-6-1
Connections:
- net VBUS is gone; now on net GND: U4.AD2 (VBUS)
- net ANT: now also L5.1
- net DEC1: now also C5.1
- net GND: now also B1.1, IC1.11 (GND_5), IC1.17 (GND_6), IC1.9 (GND_4), C1.2, C11.2, C12.2, C14.2, C15.2, C16.2, C2.2, C4.2, C5.2, C6.2, C7.2, C8.2, C9.2, L7.2, X1.2 (GND), X1.4 (GND)
- net VBATT: now also B1.2, IC1.14 (VDD_1), IC1.16 (VDD_2), C12.1, C14.1, C6.1, C7.1, C8.1, L2.2, L4.2
- net XC2: now reaches U4.A23 (XC2)
- net XC2: now also C2.1, X1.3
- net DCCH: now reaches U4.AB2 (DCCH)
- net DCCH: now also L4.1
- net XC1: now reaches U4.B24 (XC1)
- net XC1: now also C1.1, X1.1
- net DCC: now reaches U4.B3 (DCC)
- net DCC: now also L2.1
- net DEC4: now reaches U4.B5 (DEC4)
- net DEC4: now also U4.E24 (DEC6), C15.1
- new net A_conn: C4.1, L1.2, L5.2
- new net RF: L1.1, L7.3
- no-connect marks 1 -> 4
Other:
- added sheet GPSmod (GPSmod.kicad_sch)
- moved on the sheet: R1, R2, R3, SC1, SC2

Commit message: added the GPS and finished Bluetooth antennas
Parts:
- removed C17, C18: 12pF NP0 ±2%, 0402, easyeda:C0402, symbol EasyEDA:0402CG120J500NT
- added C19: 10uF, easyeda:C0603, symbol EasyEDA:CL10A106KP8NNNC
- added L3: 47nH, easyeda:L0402, symbol EasyEDA:LQW15AN47NG00D
- added U1: GPS1003, easyeda:ANT-SMD_L10.0-W3.0, symbol EasyEDA:GPS1003
- added U2: ATGM336H-5N31, easyeda:GPSM-SMD_ATGM336H-TR, symbol EasyEDA:ATGM336H-5N31
- L7: value ANT3216A063R2400A -> Bluetooth Antenna
Connections:
- net GND: now also C19.2, U2.1 (GND), U2.10 (GND), U2.12 (GND)
- net VBATT: now also C19.1, U2.6 (VBAT), U2.8 (VCC)
- net XC2: no longer X1.3
- net GPS_RX: now reaches U4.AD10 (P0.15)
- net GPS_RX: now also U2.3 (RXD)
- net 1PPS: now reaches U4.AD12 (P0.17)
- net 1PPS: now also U2.4 (1PPS)
- net On/Off: now reaches U4.AD16 (P0.20)
- net On/Off: now also U2.5 (ON/OFF)
- net GPS_TX: now reaches U4.AD8 (P0.13)
- net GPS_TX: now also U2.2 (TXD)
- new net RF_signal_G: L3.2, U1.1, U2.11 (RF_IN)
- new net VCC_RF: L3.1, U2.14 (VCC_RF)
- no-connect marks 4 -> 14
Other:
- moved on the sheet: C1, C2, IC1, L4, LS1, SC2, X1

Commit message: updated pcb and schematic
Parts:
- removed C11: 100pF NP0 ±5%, 0402, easyeda:C0402, symbol EasyEDA:0402CG101J500NT
- removed LS1: PKLCS1212E4001-R1, PKLCS1212E4001R1, symbol PKLCS1212E4001-R1:PKLCS1212E4001-R1
- added C3: 0.3pF, easyeda:C0201, symbol easyeda:GRM0335C1ER30BA01D
- added FL1: 2450LP14A100T, easyeda:FILTER-SMD_0603-6P-L1.6-W0.8_2450LP14A100T, symbol easyeda:2450LP14A100T
- C1: symbol EasyEDA:0402CG120J500NT -> easyeda:0402CG120J500NT
- C14, C15, C6: footprint GRM18x -> Capacitor_SMD:C_0603_1608Metric
- SC1, SC2: footprint (none) -> Capacitor_THT:CP_Radial_D10.0mm_P5.00mm
- U1: value GPS1003 -> GPS
Connections:
- net BATT_RAW is gone; now on net VBATT: R1.1
- net ANT: no longer IC1.10 (ANT)
- net DEC4: now also C16.1
- net GND: now also U4.B7 (VSS), C3.1, FL1.1 (GND), FL1.3 (GND), FL1.4 (GND), FL1.6 (GND); no longer IC1.1 (N/C_1)
- net RF: now also IC1.4 (TXRX); no longer L7.3
- net VBATT: no longer IC1.14 (VDD_1)
- net XC2: now also X1.3
- net DEC5: now reaches C9.1
- net DEC5: now also U4.N24 (DEC5)
- net BLUT_RX: now reaches U4.B15 (P1.14)
- net BLUT_RX: now also IC1.6 (RXEN)
- net BLUT_TX: now reaches U4.B17 (P1.12)
- net BLUT_TX: now also IC1.5 (TXEN)
- new net FILTER: C3.2, FL1.2 (IN), IC1.10 (ANT)
- new net FILTER_O: FL1.5 (OUT), L7.3
- no-connect marks 14 -> 62
Other:
- removed sheet GPSmod
- moved on the sheet: C4, L4

Commit message: updated pcb and schematic and BOM
Parts:
- removed R2, R3: 100Ω, Resistor_SMD:R_0402_1005Metric, symbol Device:R
- removed SC1: 3F,2.7V, Capacitor_THT:CP_Radial_D10.0mm_P5.00mm, symbol Device:C_Polarized
- added C10: KR-5R5C155-R, KR5R5C155R, symbol KR-5R5C155-R:KR-5R5C155-R
Connections:
- net GND: now also C10.1 (-)
- net VBATT: now also C10.2 (+); no longer B1.2, R1.1
- new net BATT_RAW: B1.2, R1.1
