File: backups/Wtracker.kicad_pcb (KiCad board)
At the start: 2 copper layers, 85.8 x 53.4 mm, 33 parts, among them IC1 RFX2401C, U1 GPS, U2 ATGM336H-5N31, U4 NRF52840-QIAA-R, X1 NX2016SA-32MHZ-STD-CZS-5

Commit message: the goat
Routing:
- net GND: track 9.31 -> 75.5 mm, vias 2 -> 13
- net /On/Off: track 22.5 -> 31.4 mm
- net /1PPS: track 20.2 -> 27.5 mm
- net /DEC4: track 40.4 -> 42.3 mm
- net /VBATT: track 144.0 -> 142.7 mm
- net /XC2: track 14.6 -> 15.5 mm
